File: 20mA_OUT.sch (KiCad schematic (older format))
At the start: 7 parts, among them Q1 IRF540N, U4 LM321

Commit message: Comments and Notation for clarity
Other:
- note added: "2nd Order Low Pass Filter"
- moved on the sheet: Q1, R10, U4
Changed lines of the file:
@@
 encoding utf-8
 Sheet 3 6
-Title ""
-Date ""
-Rev ""
-Comp ""
-Comment1 ""
+Title "PWM to 20mA Output"
+Date "2021-05-25"
+Rev "1"
+Comp "Harsch Systems"
+Comment1 "Tyler Stowell"
 Comment2 ""
 Comment3 ""
@@
 L Amplifier_Operational:LM321 U?
 U 1 1 60ABF5F3
-P 6400 3700
+P 6700 3700
 AR Path="/60A68B69/60ABF5F3" Ref="U?"  Part="1"
 AR Path="/60ABD2CD/60ABF5F3" Ref="U4"  Part="1"
-F 0 "U4" H 6744 3746 50  0000 L CNN
-F 1 "LM321" H 6744 3655 50  0000 L CNN
-F 2 "Package_TO_SOT_SMD:SOT-23-5" H 6400 3700 50  0001 C CNN
-F 3 "http://www.ti.com/lit/ds/symlink/lm321.pdf" H 6400 3700 50  0001 C CNN
-	1    6400 3700
+F 0 "U4" H 6800 3600 50  0000 L CNN
+F 1 "LM321" H 6800 3500 50  0000 L CNN
+F 2 "Package_TO_SOT_SMD:SOT-23-5" H 6700 3700 50  0001 C CNN
+F 3 "http://www.ti.com/lit/ds/symlink/lm321.pdf" H 6700 3700 50  0001 C CNN
+	1    6700 3700
 	1    0    0    -1
 $EndComp
@@
 L Device:R_US R?
 U 1 1 60ABF5FF
-P 5850 4600
+P 6150 4600
 AR Path="/60A68B69/60ABF5FF" Ref="R?"  Part="1"
 AR Path="/60ABD2CD/60ABF5FF" Ref="R10"  Part="1"
-F 0 "R10" V 5645 4600 50  0000 C CNN
-F 1 "150" V 5736 4600 50  0000 C CNN
-F 2 "" V 5890 4590 50  0001 C CNN
-F 3 "~" H 5850 4600 50  0001 C CNN
-	1    5850 4600
+F 0 "R10" V 5945 4600 50  0000 C CNN
+F 1 "150" V 6036 4600 50  0000 C CNN
+F 2 "" V 6190 4590 50  0001 C CNN
+F 3 "~" H 6150 4600 50  0001 C CNN
+	1    6150 4600
 	0    1    1    0
 $EndComp
@@
 	5500 3600 5500 3800
 Wire Wire Line
-	5500 3600 6100 3600
-Connection ~ 5500 3600
+	6400 3800 6400 4600
 Wire Wire Line
-	6100 3800 6100 4600
-Wire Wire Line
-	6100 4600 6000 4600
-Wire Wire Line
-	5700 4600 5500 4600
+	6400 4600 6300 4600
 Wire Wire Line
 	4800 4300 4800 4600
@@
 Wire Wire Line
 	5500 4300 5500 4600
-Connection ~ 5500 4600
 Wire Wire Line
 	5500 4600 4800 4600
-Text HLabel 7300 3250 2    50   Input ~ 0
+Text HLabel 7600 3250 2    50   Input ~ 0
 OUT
-Text GLabel 6500 4150 2    50   Input ~ 0
+Text GLabel 6800 4150 2    50   Input ~ 0
 GND
 Wire Wire Line
-	6300 4000 6300 4150
+	6600 4000 6600 4150
 Wire Wire Line
-	6300 4150 6500 4150
-Text GLabel 6500 3250 2    50   Input ~ 0
+	6600 4150 6800 4150
+Text GLabel 6800 3250 2    50   Input ~ 0
 24V
 Wire Wire Line
-	6300 3400 6300 3250
+	6600 3400 6600 3250
 Wire Wire Line
-	6300 3250 6500 3250
+	6600 3250 6800 3250
 $Comp
 L Transistor_FET:IRF540N Q1
 U 1 1 60AC135E
-P 7050 3700
-F 0 "Q1" H 7254 3746 50  0000 L CNN
-F 1 "IRF540N" H 7254 3655 50  0000 L CNN
-F 2 "Package_TO_SOT_THT:TO-220-3_Vertical" H 7300 3625 50  0001 L CIN
-F 3 "http://www.irf.com/product-info/datasheets/data/irf540n.pdf" H 7050 3700 50  0001 L CNN
-	1    7050 3700
+P 7350 3700
+F 0 "Q1" H 7554 3746 50  0000 L CNN
+F 1 "IRF540N" H 7554 3655 50  0000 L CNN
+F 2 "Package_TO_SOT_THT:TO-220-3_Vertical" H 7600 3625 50  0001 L CIN
+F 3 "http://www.irf.com/product-info/datasheets/data/irf540n.pdf" H 7350 3700 50  0001 L CNN
+	1    7350 3700
 	1    0    0    -1
 $EndComp
 Wire Wire Line
-	6700 3700 6850 3700
+	7000 3700 7150 3700
 Wire Wire Line
-	6100 4600 7150 4600
+	6400 4600 7450 4600
 Wire Wire Line
-	7150 4600 7150 3900
-Connection ~ 6100 4600
+	7450 4600 7450 3900
+Connection ~ 6400 4600
 Wire Wire Line
-	7150 3500 7150 3250
+	7450 3500 7450 3250
 Wire Wire Line
-	7150 3250 7300 3250
+	7450 3250 7600 3250
+Wire Wire Line
+	6000 4600 5500 4600
+Connection ~ 5500 4600
+Wire Wire Line
+	6400 3600 5500 3600
+Connection ~ 5500 3600
+Text Notes 4600 4800 0    50   ~ 0
+2nd Order Low Pass Filter
+Wire Notes Line
+	4200 4700 4200 3350
+Wire Notes Line
+	5950 4700 4200 4700
+Wire Notes Line
+	5950 3350 5950 4700
+Wire Notes Line
+	4200 3350 5950 3350
 $EndSCHEMATC

Commit message: Footprint Association
Parts:
- removed U4: LM321, Package_TO_SOT_SMD:SOT-23-5, symbol Amplifier_Operational:LM321
- added U2: LM324, Package_DIP:DIP-14_W7.62mm, symbol Amplifier_Operational:LM324
- C2: renamed from C4; footprint (none) -> Capacitor_THT:C_Disc_D5.1mm_W3.2mm_P5.00mm
- C3: renamed from C5; footprint (none) -> Capacitor_THT:C_Disc_D5.1mm_W3.2mm_P5.00mm
- R4: renamed from R8; footprint (none) -> Resistor_THT:R_Axial_DIN0207_L6.3mm_D2.5mm_P10.16mm_Horizontal
- R5: renamed from R9; footprint (none) -> Resistor_THT:R_Axial_DIN0207_L6.3mm_D2.5mm_P10.16mm_Horizontal
- R6: renamed from R10; footprint (none) -> Resistor_THT:R_Axial_DIN0207_L6.3mm_D2.5mm_P10.16mm_Horizontal
Connections:
- net at C3.1, R5.1: now also U2.5 (+)
- net at Q1.3 (S), R6.1: now also U2.6 (-)
- net at Q1.1 (G): now also U2.7
Changed lines of the file:
@@
 P 4450 3600
 AR Path="/60A68B69/60ABF5D9" Ref="R?"  Part="1"
-AR Path="/60ABD2CD/60ABF5D9" Ref="R8"  Part="1"
-F 0 "R8" V 4245 3600 50  0000 C CNN
+AR Path="/60ABD2CD/60ABF5D9" Ref="R4"  Part="1"
+F 0 "R4" V 4245 3600 50  0000 C CNN
 F 1 "2.2k" V 4336 3600 50  0000 C CNN
-F 2 "" V 4490 3590 50  0001 C CNN
+F 2 "Resistor_THT:R_Axial_DIN0207_L6.3mm_D2.5mm_P10.16mm_Horizontal" V 4490 3590 50  0001 C CNN
 F 3 "~" H 4450 3600 50  0001 C CNN
 	1    4450 3600
@@
 P 4800 4050
 AR Path="/60A68B69/60ABF5E0" Ref="C?"  Part="1"
-AR Path="/60ABD2CD/60ABF5E0" Ref="C4"  Part="1"
-F 0 "C4" H 4978 4096 50  0000 L CNN
+AR Path="/60ABD2CD/60ABF5E0" Ref="C2"  Part="1"
+F 0 "C2" H 4978 4096 50  0000 L CNN
 F 1 "2.2μ" H 4978 4005 50  0000 L CNN
-F 2 "" H 4800 4050 50  0001 C CNN
+F 2 "Capacitor_THT:C_Disc_D5.1mm_W3.2mm_P5.00mm" H 4800 4050 50  0001 C CNN
 F 3 "~" H 4800 4050 50  0001 C CNN
 	1    4800 4050
@@
 P 5150 3600
 AR Path="/60A68B69/60ABF5E6" Ref="R?"  Part="1"
-AR Path="/60ABD2CD/60ABF5E6" Ref="R9"  Part="1"
-F 0 "R9" V 4945 3600 50  0000 C CNN
+AR Path="/60ABD2CD/60ABF5E6" Ref="R5"  Part="1"
+F 0 "R5" V 4945 3600 50  0000 C CNN
 F 1 "2.2k" V 5036 3600 50  0000 C CNN
-F 2 "" V 5190 3590 50  0001 C CNN
+F 2 "Resistor_THT:R_Axial_DIN0207_L6.3mm_D2.5mm_P10.16mm_Horizontal" V 5190 3590 50  0001 C CNN
 F 3 "~" H 5150 3600 50  0001 C CNN
 	1    5150 3600
@@
 P 5500 4050
 AR Path="/60A68B69/60ABF5EC" Ref="C?"  Part="1"
-AR Path="/60ABD2CD/60ABF5EC" Ref="C5"  Part="1"
-F 0 "C5" H 5678 4096 50  0000 L CNN
+AR Path="/60ABD2CD/60ABF5EC" Ref="C3"  Part="1"
+F 0 "C3" H 5678 4096 50  0000 L CNN
 F 1 "2.2μ" H 5678 4005 50  0000 L CNN
-F 2 "" H 5500 4050 50  0001 C CNN
+F 2 "Capacitor_THT:C_Disc_D5.1mm_W3.2mm_P5.00mm" H 5500 4050 50  0001 C CNN
 F 3 "~" H 5500 4050 50  0001 C CNN
 	1    5500 4050
@@
 GND
 $Comp
-L Amplifier_Operational:LM321 U?
-U 1 1 60ABF5F3
-P 6700 3700
-AR Path="/60A68B69/60ABF5F3" Ref="U?"  Part="1"
-AR Path="/60ABD2CD/60ABF5F3" Ref="U4"  Part="1"
-F 0 "U4" H 6800 3600 50  0000 L CNN
-F 1 "LM321" H 6800 3500 50  0000 L CNN
-F 2 "Package_TO_SOT_SMD:SOT-23-5" H 6700 3700 50  0001 C CNN
-F 3 "http://www.ti.com/lit/ds/symlink/lm321.pdf" H 6700 3700 50  0001 C CNN
-	1    6700 3700
-	1    0    0    -1
-$EndComp
-$Comp
 L Device:R_US R?
 U 1 1 60ABF5FF
 P 6150 4600
 AR Path="/60A68B69/60ABF5FF" Ref="R?"  Part="1"
-AR Path="/60ABD2CD/60ABF5FF" Ref="R10"  Part="1"
-F 0 "R10" V 5945 4600 50  0000 C CNN
+AR Path="/60ABD2CD/60ABF5FF" Ref="R6"  Part="1"
+F 0 "R6" V 5945 4600 50  0000 C CNN
 F 1 "150" V 6036 4600 50  0000 C CNN
-F 2 "" V 6190 4590 50  0001 C CNN
+F 2 "Resistor_THT:R_Axial_DIN0207_L6.3mm_D2.5mm_P10.16mm_Horizontal" V 6190 4590 50  0001 C CNN
 F 3 "~" H 6150 4600 50  0001 C CNN
 	1    6150 4600
@@
 Text HLabel 7600 3250 2    50   Input ~ 0
 OUT
-Text GLabel 6800 4150 2    50   Input ~ 0
-GND
-Wire Wire Line
-	6600 4000 6600 4150
-Wire Wire Line
-	6600 4150 6800 4150
-Text GLabel 6800 3250 2    50   Input ~ 0
-24V
-Wire Wire Line
-	6600 3400 6600 3250
-Wire Wire Line
-	6600 3250 6800 3250
 $Comp
 L Transistor_FET:IRF540N Q1
@@
 Wire Wire Line
 	7000 3700 7150 3700
-Wire Wire Line
-	6400 4600 7450 4600
 Wire Wire Line
 	7450 4600 7450 3900
@@
 Wire Notes Line
 	4200 3350 5950 3350
+Wire Wire Line
+	6400 4600 7450 4600
+$Comp
+L Amplifier_Operational:LM324 U2
+U 2 1 60C66065
+P 6700 3700
+F 0 "U2" H 6700 4067 50  0000 C CNN
+F 1 "LM324" H 6700 3976 50  0000 C CNN
+F 2 "Package_DIP:DIP-14_W7.62mm" H 6650 3800 50  0001 C CNN
+F 3 "http://www.ti.com/lit/ds/symlink/lm2902-n.pdf" H 6750 3900 50  0001 C CNN
+	2    6700 3700
+	1    0    0    -1
+$EndComp
 $EndSCHEMATC

Commit message: Fixed a couple of discrepancies between my test circuit and the schematic
Parts:
- added R27: 10, Resistor_THT:R_Axial_DIN0207_L6.3mm_D2.5mm_P10.16mm_Horizontal, symbol Device:R_US
- Q1: value IRF540N -> IRF510N
Connections:
- net at Q1.1 (G): now also R27.1; no longer U2.7
- new net: R27.2, U2.7
Other:
- moved on the sheet: Q1
Changed lines of the file:
@@
 Wire Wire Line
 	5500 4600 4800 4600
-Text HLabel 7600 3250 2    50   Input ~ 0
+Text HLabel 7850 3250 2    50   Input ~ 0
 OUT
 $Comp
 L Transistor_FET:IRF540N Q1
 U 1 1 60AC135E
-P 7350 3700
-F 0 "Q1" H 7554 3746 50  0000 L CNN
-F 1 "IRF540N" H 7554 3655 50  0000 L CNN
-F 2 "Package_TO_SOT_THT:TO-220-3_Vertical" H 7600 3625 50  0001 L CIN
-F 3 "http://www.irf.com/product-info/datasheets/data/irf540n.pdf" H 7350 3700 50  0001 L CNN
-	1    7350 3700
+P 7600 3700
+F 0 "Q1" H 7804 3746 50  0000 L CNN
+F 1 "IRF510N" H 7804 3655 50  0000 L CNN
+F 2 "Package_TO_SOT_THT:TO-220-3_Vertical" H 7850 3625 50  0001 L CIN
+F 3 "http://www.irf.com/product-info/datasheets/data/irf540n.pdf" H 7600 3700 50  0001 L CNN
+	1    7600 3700
 	1    0    0    -1
 $EndComp
 Wire Wire Line
-	7000 3700 7150 3700
+	7700 4600 7700 3900
 Wire Wire Line
-	7450 4600 7450 3900
-Connection ~ 6400 4600
+	7700 3500 7700 3250
 Wire Wire Line
-	7450 3500 7450 3250
-Wire Wire Line
-	7450 3250 7600 3250
+	7700 3250 7850 3250
 Wire Wire Line
 	6000 4600 5500 4600
@@
 Wire Notes Line
 	4200 3350 5950 3350
-Wire Wire Line
-	6400 4600 7450 4600
 $Comp
 L Amplifier_Operational:LM324 U2
@@
 	1    0    0    -1
 $EndComp
+$Comp
+L Device:R_US R?
+U 1 1 60C85CA5
+P 7200 3700
+AR Path="/60A68B69/60C85CA5" Ref="R?"  Part="1"
+AR Path="/60ABD2CD/60C85CA5" Ref="R27"  Part="1"
+F 0 "R27" V 6995 3700 50  0000 C CNN
+F 1 "10" V 7086 3700 50  0000 C CNN
+F 2 "Resistor_THT:R_Axial_DIN0207_L6.3mm_D2.5mm_P10.16mm_Horizontal" V 7240 3690 50  0001 C CNN
+F 3 "~" H 7200 3700 50  0001 C CNN
+	1    7200 3700
+	0    1    1    0
+$EndComp
+Wire Wire Line
+	7000 3700 7050 3700
+Wire Wire Line
+	7350 3700 7400 3700
+Wire Wire Line
+	7700 4600 6400 4600
+Connection ~ 6400 4600
 $EndSCHEMATC

Commit message: Finished 1st revision of 24V digital output circuit
Parts:
- renumbered R27 to R7
Changed lines of the file:
@@
 P 7200 3700
 AR Path="/60A68B69/60C85CA5" Ref="R?"  Part="1"
-AR Path="/60ABD2CD/60C85CA5" Ref="R27"  Part="1"
-F 0 "R27" V 6995 3700 50  0000 C CNN
+AR Path="/60ABD2CD/60C85CA5" Ref="R7"  Part="1"
+F 0 "R7" V 6995 3700 50  0000 C CNN
 F 1 "10" V 7086 3700 50  0000 C CNN
 F 2 "Resistor_THT:R_Axial_DIN0207_L6.3mm_D2.5mm_P10.16mm_Horizontal" V 7240 3690 50  0001 C CNN
