File: DIG_IN.sch (KiCad schematic (older format))
At the start: 12 parts, among them U5 PC817, U6 PC817

Commit message: Finished 1st revision of 24V digital output circuit
Parts:
- removed D3: D, Diode_THT:D_A-405_P10.16mm_Horizontal, symbol Device:D
- removed D?: LED, LED_THT:LED_D5.0mm, symbol Device:LED
- removed R17: 4.7k, Resistor_THT:R_Axial_DIN0207_L6.3mm_D2.5mm_P10.16mm_Horizontal, symbol Device:R_US
- removed R? (x2): 4.7k, symbol Device:R_US
- added D1: D, Diode_THT:D_A-405_P10.16mm_Horizontal, symbol Device:D
- added D3: LED, LED_THT:LED_D5.0mm, symbol Device:LED
- added R18: 4.7k, Resistor_THT:R_Axial_DIN0207_L6.3mm_D2.5mm_P10.16mm_Horizontal, symbol Device:R_US
- gave numbers to parts that had none: 2
- renumbered D4 to D2, R19 to R20, R20 to R21
Connections:
- net IN+1: now also D1.1 (K), D3.2 (A); no longer U5.1
- net IN+2: no longer U6.1
- net IN-1: now also R18.1
- net at U5.2: now also D1.2 (A), R18.2
- net at D4.1 (K): now also U6.1
- new net: D3.1 (K), U5.1
Other:
- moved on the sheet: D2, D4, R19
Changed lines of the file:
@@
 Wire Wire Line
 	5400 3900 5400 3550
-$Comp
-L Device:R_US R17
-U 1 1 60B3319D
-P 4950 3900
-F 0 "R17" V 5155 3900 50  0000 C CNN
-F 1 "4.7k" V 5064 3900 50  0000 C CNN
-F 2 "Resistor_THT:R_Axial_DIN0207_L6.3mm_D2.5mm_P10.16mm_Horizontal" V 4990 3890 50  0001 C CNN
-F 3 "~" H 4950 3900 50  0001 C CNN
-	1    4950 3900
-	0    -1   -1   0
-$EndComp
 Text GLabel 6050 3600 3    50   Input ~ 0
 GND
 $Comp
-L Device:R_US R19
+L Device:R_US R20
 U 1 1 60B348C0
 P 6550 3350
-F 0 "R19" V 6345 3350 50  0000 C CNN
+F 0 "R20" V 6345 3350 50  0000 C CNN
 F 1 "20k" V 6436 3350 50  0000 C CNN
 F 2 "Resistor_THT:R_Axial_DIN0207_L6.3mm_D2.5mm_P10.16mm_Horizontal" V 6590 3340 50  0001 C CNN
@@
 Text Notes 6400 2900 0    50   ~ 0
 Pull Up Resistor
-$Comp
-L Device:D D3
-U 1 1 60B8ECB5
-P 5200 3450
-F 0 "D3" V 5154 3530 50  0000 L CNN
-F 1 "D" V 5245 3530 50  0000 L CNN
-F 2 "Diode_THT:D_A-405_P10.16mm_Horizontal" H 5200 3450 50  0001 C CNN
-F 3 "~" H 5200 3450 50  0001 C CNN
-	1    5200 3450
-	0    1    1    0
-$EndComp
-Wire Wire Line
-	5400 3900 5200 3900
-Wire Wire Line
-	5200 3600 5200 3900
-Wire Wire Line
-	5200 3300 5200 3000
-Wire Wire Line
-	5200 3000 5400 3000
 Text HLabel 4400 4300 0    50   Input ~ 0
 IN+2
@@
 GND
 $Comp
-L Device:R_US R20
+L Device:R_US R21
 U 1 1 60B9B8D8
 P 6550 4650
-F 0 "R20" V 6345 4650 50  0000 C CNN
+F 0 "R21" V 6345 4650 50  0000 C CNN
 F 1 "20k" V 6436 4650 50  0000 C CNN
 F 2 "Resistor_THT:R_Axial_DIN0207_L6.3mm_D2.5mm_P10.16mm_Horizontal" V 6590 4640 50  0001 C CNN
@@
 Pull Up Resistor
 $Comp
-L Device:D D4
+L Device:D D2
 U 1 1 60B9B8F3
-P 5200 4750
-F 0 "D4" V 5154 4830 50  0000 L CNN
-F 1 "D" V 5245 4830 50  0000 L CNN
-F 2 "Diode_THT:D_A-405_P10.16mm_Horizontal" H 5200 4750 50  0001 C CNN
-F 3 "~" H 5200 4750 50  0001 C CNN
-	1    5200 4750
-	0    1    1    0
-$EndComp
-Wire Wire Line
-	5400 5200 5200 5200
-Wire Wire Line
-	5200 4900 5200 5200
-Wire Wire Line
-	5200 4600 5200 4300
-Wire Wire Line
-	5200 4300 5400 4300
-$Comp
-L Device:LED D?
-U 1 1 60C8AFD4
-P 4700 3300
-F 0 "D?" V 4750 3150 50  0000 C CNN
-F 1 "LED" V 4650 3150 50  0000 C CNN
-F 2 "LED_THT:LED_D5.0mm" H 4700 3300 50  0001 C CNN
-F 3 "~" H 4700 3300 50  0001 C CNN
-	1    4700 3300
+P 4900 4750
+F 0 "D2" V 4854 4830 50  0000 L CNN
+F 1 "D" V 4945 4830 50  0000 L CNN
+F 2 "Diode_THT:D_A-405_P10.16mm_Horizontal" H 4900 4750 50  0001 C CNN
+F 3 "~" H 4900 4750 50  0001 C CNN
+	1    4900 4750
+	0    1    1    0
+$EndComp
+$Comp
+L Device:R_US R19
+U 1 1 60CA13C5
+P 4650 5200
+F 0 "R19" V 4855 5200 50  0000 C CNN
+F 1 "4.7k" V 4764 5200 50  0000 C CNN
+F 2 "Resistor_THT:R_Axial_DIN0207_L6.3mm_D2.5mm_P10.16mm_Horizontal" V 4690 5190 50  0001 C CNN
+F 3 "~" H 4650 5200 50  0001 C CNN
+	1    4650 5200
 	0    -1   -1   0
 $EndComp
-Text Notes 4100 3350 0    50   ~ 0
+$Comp
+L Device:LED D4
+U 1 1 60CA13CB
+P 5150 4300
+F 0 "D4" H 5150 4100 50  0000 C CNN
+F 1 "LED" H 5150 4200 50  0000 C CNN
+F 2 "LED_THT:LED_D5.0mm" H 5150 4300 50  0001 C CNN
+F 3 "~" H 5150 4300 50  0001 C CNN
+	1    5150 4300
+	-1   0    0    1
+$EndComp
+Wire Notes Line
+	5350 4450 5350 4050
+Wire Notes Line
+	4950 4050 4950 4450
+Wire Notes Line
+	4950 4450 5350 4450
+Wire Notes Line
+	5350 4050 4950 4050
+Text Notes 5350 4550 2    50   ~ 0
 Status LED
-Wire Notes Line
-	4550 3500 4950 3500
-Wire Notes Line
-	4950 3100 4550 3100
-Wire Notes Line
-	4550 3100 4550 3500
-Wire Notes Line
-	4950 3500 4950 3100
-Connection ~ 5200 3000
-Wire Wire Line
-	4400 3000 4700 3000
-$Comp
-L Device:R_US R?
-U 1 1 60C967CD
-P 4700 3700
-F 0 "R?" H 4500 3750 50  0000 L CNN
-F 1 "4.7k" H 4450 3650 50  0000 L CNN
-F 2 "" V 4740 3690 50  0001 C CNN
-F 3 "~" H 4700 3700 50  0001 C CNN
-	1    4700 3700
-	1    0    0    -1
-$EndComp
-Wire Wire Line
-	4700 3000 4700 3150
-Connection ~ 4700 3000
-Wire Wire Line
-	4700 3000 5200 3000
-Wire Wire Line
-	4700 3450 4700 3550
-Wire Wire Line
-	4400 3900 4700 3900
-Wire Wire Line
-	4700 3850 4700 3900
-Connection ~ 4700 3900
-Wire Wire Line
-	4700 3900 4800 3900
-Wire Wire Line
-	5100 3900 5200 3900
-Connection ~ 5200 3900
-$Comp
-L Device:R_US R?
-U 1 1 60CA13C5
-P 4950 5200
-F 0 "R?" V 5155 5200 50  0000 C CNN
-F 1 "4.7k" V 5064 5200 50  0000 C CNN
-F 2 "Resistor_THT:R_Axial_DIN0207_L6.3mm_D2.5mm_P10.16mm_Horizontal" V 4990 5190 50  0001 C CNN
-F 3 "~" H 4950 5200 50  0001 C CNN
-	1    4950 5200
+Wire Wire Line
+	4400 4300 4900 4300
+Wire Wire Line
+	5300 4300 5400 4300
+Wire Wire Line
+	5400 5200 4900 5200
+Wire Wire Line
+	4900 4900 4900 5200
+Connection ~ 4900 5200
+Wire Wire Line
+	4900 5200 4800 5200
+Wire Wire Line
+	4500 5200 4400 5200
+Wire Wire Line
+	4900 4600 4900 4300
+Connection ~ 4900 4300
+Wire Wire Line
+	4900 4300 5000 4300
+$Comp
+L Device:D D1
+U 1 1 60CF166B
+P 4900 3450
+F 0 "D1" V 4854 3530 50  0000 L CNN
+F 1 "D" V 4945 3530 50  0000 L CNN
+F 2 "Diode_THT:D_A-405_P10.16mm_Horizontal" H 4900 3450 50  0001 C CNN
+F 3 "~" H 4900 3450 50  0001 C CNN
+	1    4900 3450
+	0    1    1    0
+$EndComp
+$Comp
+L Device:R_US R18
+U 1 1 60CF1671
+P 4650 3900
+F 0 "R18" V 4855 3900 50  0000 C CNN
+F 1 "4.7k" V 4764 3900 50  0000 C CNN
+F 2 "Resistor_THT:R_Axial_DIN0207_L6.3mm_D2.5mm_P10.16mm_Horizontal" V 4690 3890 50  0001 C CNN
+F 3 "~" H 4650 3900 50  0001 C CNN
+	1    4650 3900
 	0    -1   -1   0
 $EndComp
 $Comp
-L Device:LED D?
-U 1 1 60CA13CB
-P 4700 4600
-F 0 "D?" V 4750 4450 50  0000 C CNN
-F 1 "LED" V 4650 4450 50  0000 C CNN
-F 2 "LED_THT:LED_D5.0mm" H 4700 4600 50  0001 C CNN
-F 3 "~" H 4700 4600 50  0001 C CNN
-	1    4700 4600
-	0    -1   -1   0
-$EndComp
-Wire Notes Line
-	4550 4800 4950 4800
-Wire Notes Line
-	4950 4400 4550 4400
-Wire Notes Line
-	4550 4400 4550 4800
-Wire Notes Line
-	4950 4800 4950 4400
-Wire Wire Line
-	4400 4300 4700 4300
-$Comp
-L Device:R_US R?
-U 1 1 60CA13D6
-P 4700 5000
-F 0 "R?" H 4500 5050 50  0000 L CNN
-F 1 "4.7k" H 4450 4950 50  0000 L CNN
-F 2 "" V 4740 4990 50  0001 C CNN
-F 3 "~" H 4700 5000 50  0001 C CNN
-	1    4700 5000
-	1    0    0    -1
-$EndComp
-Wire Wire Line
-	4700 4300 4700 4450
-Connection ~ 4700 4300
-Wire Wire Line
-	4700 4300 5200 4300
-Wire Wire Line
-	4700 4750 4700 4850
-Wire Wire Line
-	4400 5200 4700 5200
-Wire Wire Line
-	4700 5150 4700 5200
-Connection ~ 4700 5200
-Wire Wire Line
-	4700 5200 4800 5200
-Wire Wire Line
-	5100 5200 5200 5200
-Connection ~ 5200 5200
-Text Notes 4100 4650 0    50   ~ 0
+L Device:LED D3
+U 1 1 60CF1677
+P 5150 3000
+F 0 "D3" H 5150 2800 50  0000 C CNN
+F 1 "LED" H 5150 2900 50  0000 C CNN
+F 2 "LED_THT:LED_D5.0mm" H 5150 3000 50  0001 C CNN
+F 3 "~" H 5150 3000 50  0001 C CNN
+	1    5150 3000
+	-1   0    0    1
+$EndComp
+Wire Notes Line
+	5350 3150 5350 2750
+Wire Notes Line
+	4950 2750 4950 3150
+Wire Notes Line
+	4950 3150 5350 3150
+Wire Notes Line
+	5350 2750 4950 2750
+Text Notes 5350 3250 2    50   ~ 0
 Status LED
+Wire Wire Line
+	4400 3000 4900 3000
+Wire Wire Line
+	5300 3000 5400 3000
+Wire Wire Line
+	5400 3900 4900 3900
+Wire Wire Line
+	4900 3600 4900 3900
+Connection ~ 4900 3900
+Wire Wire Line
+	4900 3900 4800 3900
+Wire Wire Line
+	4500 3900 4400 3900
+Wire Wire Line
+	4900 3300 4900 3000
+Connection ~ 4900 3000
+Wire Wire Line
+	4900 3000 5000 3000
 $EndSCHEMATC
