File: RP2040_Board.sch (KiCad schematic (older format))
At the start: 9 parts, among them J1 V_OUT, J2 mA_OUT, J3 DIG_IN, J4 DIG_IN, J5 DIG_OUT, J6 DIG_OUT, J7 mA_IN, J8 V_IN, U1 Pico

Commit message: Cleanup and ERC compliance. Probably ready for Pcbnew after footprint association is done.
Parts:
- added J9: GND-24V, symbol Connector:Conn_01x02_Female
Connections:
- net GND: now also U1.23 (GND), J9.1 (Pin_1); no longer J2.1 (Pin_1), U1.42 (GND)
- new net 24V: J2.1 (Pin_1), J9.2 (Pin_2)
Changed lines of the file:
@@
 F3 "IN" I R 7650 4400 50
 $EndSheet
-Text GLabel 5900 5350 3    50   Input ~ 0
+Text GLabel 6700 4850 2    50   Input ~ 0
 GND
 $Sheet
@@
 NoConn ~ 6600 4550
 NoConn ~ 6600 4750
-NoConn ~ 6600 4850
 NoConn ~ 6600 4950
 NoConn ~ 6000 5250
@@
 	4150 4600 4000 4600
 Text GLabel 3950 3700 3    50   Input ~ 0
-GND
+24V
 Text GLabel 3950 2900 3    50   Input ~ 0
 GND
@@
 Wire Wire Line
 	3950 3650 3900 3650
-Wire Wire Line
-	5900 5350 5900 5250
 Text GLabel 7850 4500 3    50   Input ~ 0
 GND
@@
 Wire Wire Line
 	4050 5400 4050 5100
+Text GLabel 7800 5100 0    50   Input ~ 0
+GND
+Text GLabel 7800 5300 0    50   Input ~ 0
+24V
+$Comp
+L Connector:Conn_01x02_Female J9
+U 1 1 60B60AD3
+P 8100 5150
+F 0 "J9" H 8128 5126 50  0000 L CNN
+F 1 "GND-24V" H 8128 5035 50  0000 L CNN
+F 2 "" H 8100 5150 50  0001 C CNN
+F 3 "~" H 8100 5150 50  0001 C CNN
+	1    8100 5150
+	1    0    0    -1
+$EndComp
+Wire Wire Line
+	7800 5100 7850 5100
+Wire Wire Line
+	7850 5100 7850 5150
+Wire Wire Line
+	7850 5150 7900 5150
+Wire Wire Line
+	7800 5300 7850 5300
+Wire Wire Line
+	7850 5300 7850 5250
+Wire Wire Line
+	7850 5250 7900 5250
+Wire Wire Line
+	6600 4850 6700 4850
+NoConn ~ 5900 5250
 $EndSCHEMATC

Commit message: Finished component association
Parts:
- J1, J2, J3, J4, J5, J6, J7, J8, J9: footprint (none) -> Connector_PinHeader_1.00mm:PinHeader_1x02_P1.00mm_Vertical
Changed lines of the file:
@@
 F 0 "J7" H 8128 3526 50  0000 L CNN
 F 1 "mA_IN" H 8128 3435 50  0000 L CNN
-F 2 "" H 8100 3550 50  0001 C CNN
+F 2 "Connector_PinHeader_1.00mm:PinHeader_1x02_P1.00mm_Vertical" H 8100 3550 50  0001 C CNN
 F 3 "~" H 8100 3550 50  0001 C CNN
 	1    8100 3550
@@
 F 0 "J8" H 8128 4326 50  0000 L CNN
 F 1 "V_IN" H 8128 4235 50  0000 L CNN
-F 2 "" H 8100 4350 50  0001 C CNN
+F 2 "Connector_PinHeader_1.00mm:PinHeader_1x02_P1.00mm_Vertical" H 8100 4350 50  0001 C CNN
 F 3 "~" H 8100 4350 50  0001 C CNN
 	1    8100 4350
@@
 F 0 "J1" H 3592 2525 50  0000 C CNN
 F 1 "V_OUT" H 3592 2616 50  0000 C CNN
-F 2 "" H 3700 2850 50  0001 C CNN
+F 2 "Connector_PinHeader_1.00mm:PinHeader_1x02_P1.00mm_Vertical" H 3700 2850 50  0001 C CNN
 F 3 "~" H 3700 2850 50  0001 C CNN
 	1    3700 2850
@@
 F 0 "J2" H 3592 3325 50  0000 C CNN
 F 1 "mA_OUT" H 3592 3416 50  0000 C CNN
-F 2 "" H 3700 3650 50  0001 C CNN
+F 2 "Connector_PinHeader_1.00mm:PinHeader_1x02_P1.00mm_Vertical" H 3700 3650 50  0001 C CNN
 F 3 "~" H 3700 3650 50  0001 C CNN
 	1    3700 3650
@@
 F 0 "J3" H 3692 3975 50  0000 C CNN
 F 1 "DIG_IN" H 3692 4066 50  0000 C CNN
-F 2 "" H 3800 4300 50  0001 C CNN
+F 2 "Connector_PinHeader_1.00mm:PinHeader_1x02_P1.00mm_Vertical" H 3800 4300 50  0001 C CNN
 F 3 "~" H 3800 4300 50  0001 C CNN
 	1    3800 4300
@@
 F 0 "J4" H 3700 4650 50  0000 C CNN
 F 1 "DIG_IN" H 3700 4750 50  0000 C CNN
-F 2 "" H 3800 4600 50  0001 C CNN
+F 2 "Connector_PinHeader_1.00mm:PinHeader_1x02_P1.00mm_Vertical" H 3800 4600 50  0001 C CNN
 F 3 "~" H 3800 4600 50  0001 C CNN
 	1    3800 4600
@@
 F 0 "J5" H 3950 5000 50  0000 C CNN
 F 1 "DIG_OUT" H 3950 5100 50  0000 C CNN
-F 2 "" H 3800 5100 50  0001 C CNN
+F 2 "Connector_PinHeader_1.00mm:PinHeader_1x02_P1.00mm_Vertical" H 3800 5100 50  0001 C CNN
 F 3 "~" H 3800 5100 50  0001 C CNN
 	1    3800 5100
@@
 F 0 "J6" H 3700 5500 50  0000 C CNN
 F 1 "DIG_OUT" H 3700 5600 50  0000 C CNN
-F 2 "" H 3800 5400 50  0001 C CNN
+F 2 "Connector_PinHeader_1.00mm:PinHeader_1x02_P1.00mm_Vertical" H 3800 5400 50  0001 C CNN
 F 3 "~" H 3800 5400 50  0001 C CNN
 	1    3800 5400
@@
 F 0 "J9" H 8128 5126 50  0000 L CNN
 F 1 "GND-24V" H 8128 5035 50  0000 L CNN
-F 2 "" H 8100 5150 50  0001 C CNN
+F 2 "Connector_PinHeader_1.00mm:PinHeader_1x02_P1.00mm_Vertical" H 8100 5150 50  0001 C CNN
 F 3 "~" H 8100 5150 50  0001 C CNN
 	1    8100 5150
