File: RP2040_Board.kicad_pcb (KiCad board)
At the start: 2 copper layers, 60 parts, among them J1 V_OUT, J10 24V DC Power, J2 mA_OUT, J7 mA_IN, J8 V_IN, J9 GND-24V, Q1 IRF510N, Q2 BC337, Q3 BC337, U1 Pico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

Commit message: More PCB design work
Parts:
- removed J1: V_OUT, Connector_PinSocket_2.54mm:PinSocket_1x02_P2.54mm_Vertical
- removed J8: V_IN, Connector_PinSocket_2.54mm:PinSocket_1x02_P2.54mm_Vertical
- added ADC0: V_IN, Connector_PinSocket_2.54mm:PinSocket_1x02_P2.54mm_Vertical, F.Cu at (120.0, 77.5)
- added GP0: V_OUT, Connector_PinSocket_2.54mm:PinSocket_1x02_P2.54mm_Vertical, F.Cu at (116.2, 74.9)
- moved R10 98.7 mm to (120.0, 103.5), turned to 90 degrees
- moved C1 94.4 mm to (116.2, 100.3), turned to 90 degrees
- moved R11 88.8 mm to (123.8, 92.7), turned to 270 degrees
- moved C5 88.2 mm to (134.0, 97.8), turned to 270 degrees
- moved C4 85.7 mm to (134.0, 110.5), turned to 90 degrees
- moved R2 83.2 mm to (116.2, 90.8), turned to 90 degrees
- moved R9 81.3 mm to (130.2, 92.7), turned to 270 degrees
- moved Q1 81.3 mm to (135.3, 75.6), turned to 180 degrees
- moved R1 78.0 mm to (120.0, 90.8), turned to 90 degrees
- moved R8 74.8 mm to (130.2, 108.0), turned to 180 degrees
- moved R3 70.3 mm to (127.0, 102.9), turned to 90 degrees
- moved J10 62.2 mm to (156.2, 120.7), turned to 90 degrees
- moved U2 60.8 mm to (123.8, 90.2), turned to 90 degrees
- moved U1 56.7 mm to (102.9, 123.2), turned to 270 degrees
- moved J7 56.2 mm to (146.7, 74.9)
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Routing:
- net GND: track 58.0 -> 122.5 mm
- net /Digital Output/IN1: track 0.00 -> 60.1 mm
- net /Digital Output/IN2: track 0.00 -> 53.4 mm
- net /10V to 3.3V Input/OUT: track 0.00 -> 52.3 mm
- net Net-(R1-Pad1): track 0.00 -> 21.4 mm, vias 0 -> 1
- net /Digital Input/OUT2: track 4.34 -> 24.5 mm
- net Net-(R10-Pad1): track 0.00 -> 17.8 mm
- net Net-(Q1-Pad3): track 0.00 -> 17.2 mm
- net /PWM to 10V Output/OUT: track 0.00 -> 15.9 mm
- net Net-(R3-Pad2): track 0.00 -> 13.5 mm
- net /PWM to 10V Output/PWM: track 0.00 -> 11.1 mm
- net /PWM to 20mA Output/OUT: track 0.00 -> 10.9 mm
- net /Digital Input/OUT1: track 4.34 -> 14.3 mm
- net Net-(C4-Pad1): track 0.00 -> 9.94 mm
- net Net-(C5-Pad1): track 0.00 -> 9.72 mm
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Other:
- board text added: "IN"
- board text added: "OUT"
